File: src/Solder.kicad_sch (KiCad schematic)
At the start: 6 parts, among them SW1 SW_Push

Commit message: Add decoration
Parts:
- added RV1: R_Potentiometer, Potentiometer_THT:Potentiometer_Vishay_T73YP_Vertical, symbol Device:R_Potentiometer
Connections:
- net at D1.2 (A), D2.2 (A): now also RV1.1, RV1.3; no longer SW1.2
- new net: RV1.2, SW1.2
Changed lines of the file:
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@@
 	(paper "A4")
+	(junction
+		(at 127 90.17)
+		(diameter 0)
+		(color 0 0 0 0)
+	)
 	(junction
 		(at 127 63.5)
@@
 	)
 	(junction
-		(at 127 90.17)
+		(at 127 67.31)
 		(diameter 0)
 		(color 0 0 0 0)
@@
 	(wire
 		(pts
+			(xy 115.57 63.5) (xy 118.11 63.5)
+		)
+		(stroke
+			(width 0)
+			(type default)
+		)
+	)
+	(wire
+		(pts
 			(xy 105.41 73.66) (xy 105.41 63.5)
 		)
@@
 	(wire
 		(pts
+			(xy 121.92 67.31) (xy 127 67.31)
+		)
+		(stroke
+			(width 0)
+			(type default)
+		)
+	)
+	(wire
+		(pts
 			(xy 127 90.17) (xy 105.41 90.17)
 		)
@@
 	(wire
 		(pts
-			(xy 115.57 63.5) (xy 127 63.5)
+			(xy 127 59.69) (xy 127 63.5)
+		)
+		(stroke
+			(width 0)
+			(type default)
+		)
+	)
+	(wire
+		(pts
+			(xy 121.92 59.69) (xy 127 59.69)
 		)
 		(stroke
@@
 		)
 	)
+	(symbol
+		(lib_id "Device:R_Potentiometer")
+		(at 121.92 63.5 180)
+		(unit 1)
+		(exclude_from_sim no)
+		(in_bom yes)
+		(on_board yes)
+		(dnp no)
+		(fields_autoplaced yes)
+		(property "Reference" "RV1"
+			(at 124.46 62.2299 0)
+			(effects
+				(font
+					(size 1.27 1.27)
+				)
+				(justify right)
+			)
+		)
+		(property "Value" "R_Potentiometer"
+			(at 124.46 64.7699 0)
+			(effects
+				(font
+					(size 1.27 1.27)
+				)
+				(justify right)
+			)
+		)
+		(property "Footprint" "Potentiometer_THT:Potentiometer_Vishay_T73YP_Vertical"
+			(at 121.92 63.5 0)
+			(effects
+				(font
+					(size 1.27 1.27)
+				)
+				(hide yes)
+			)
+		)
+		(property "Datasheet" "~"
+			(at 121.92 63.5 0)
+			(effects
+				(font
+					(size 1.27 1.27)
+				)
+				(hide yes)
+			)
+		)
+		(property "Description" "Potentiometer"
+			(at 121.92 63.5 0)
+			(effects
+				(font
+					(size 1.27 1.27)
+				)
+				(hide yes)
+			)
+		)
+		(pin "2"
+		)
+		(pin "3"
+		)
+		(pin "1"
+		)
+		(instances
+			(project ""
+				(path "/8b732828-8244-451f-9bdb-50d32063189d"
+					(reference "RV1")
+					(unit 1)
+				)
+			)
+		)
+	)
