File: src/Solder.kicad_pcb (KiCad board)
At the start: 2 copper layers, 135.9 x 275.4 mm, 11 parts, among them SW1 SW_Push

Commit message: Fix potentiometer wiring
Connections:
- RV1 pad 1: Net-(D1-A) -> Net-(RV1-Pad1)
- RV1 pad 2: Net-(RV1-Pad2) -> Net-(D1-A)
- RV1 pad 3: Net-(D1-A) -> Net-(BT1--)
- SW1 pad 2: Net-(RV1-Pad2) -> Net-(RV1-Pad1)
Routing:
- net Net-(BT1--): track 30.4 -> 52.7 mm
- net Net-(RV1-Pad1): track 0.00 -> 12.8 mm
- net Net-(RV1-Pad2): track 11.4 -> 0.00 mm
- net Net-(D1-A): track 21.3 -> 24.9 mm
- net Net-(BT1-+): track 53.9 -> 52.4 mm
Changed lines of the file:
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@@
 	(net 4 "Net-(D2-K)")
 	(net 5 "Net-(D1-A)")
-	(net 6 "Net-(RV1-Pad2)")
+	(net 6 "Net-(RV1-Pad1)")
 	(footprint "LED_THT:LED_D5.0mm"
 		(layer "F.Cu")
@@
 			(layers "*.Cu" "*.Mask")
 			(remove_unused_layers no)
-			(net 5 "Net-(D1-A)")
+			(net 6 "Net-(RV1-Pad1)")
 			(pinfunction "1")
 			(pintype "passive")
@@
 			(layers "*.Cu" "*.Mask")
 			(remove_unused_layers no)
-			(net 6 "Net-(RV1-Pad2)")
+			(net 5 "Net-(D1-A)")
 			(pinfunction "2")
 			(pintype "passive")
@@
 			(layers "*.Cu" "*.Mask")
 			(remove_unused_layers no)
-			(net 5 "Net-(D1-A)")
+			(net 1 "Net-(BT1--)")
 			(pinfunction "3")
 			(pintype "passive")
@@
 			(layers "*.Cu" "*.Mask")
 			(remove_unused_layers no)
-			(net 6 "Net-(RV1-Pad2)")
+			(net 6 "Net-(RV1-Pad1)")
 			(pinfunction "2")
 			(pintype "passive")
@@
 			(layers "*.Cu" "*.Mask")
 			(remove_unused_layers no)
-			(net 6 "Net-(RV1-Pad2)")
+			(net 6 "Net-(RV1-Pad1)")
 			(pinfunction "2")
 			(pintype "passive")
@@
 	)
 	(segment
-		(start 119.37 51.25)
-		(end 121.985 51.25)
+		(start 121.985 51.25)
+		(end 130.75 60.015)
 		(width 0.2)
 		(layer "F.Cu")
@@
 	)
 	(segment
-		(start 119.37 69.75)
-		(end 121.015 69.75)
+		(start 111.940001 58.679999)
+		(end 101.219999 58.679999)
 		(width 0.2)
 		(layer "F.Cu")
@@
 	)
 	(segment
-		(start 121.985 51.25)
-		(end 130.75 60.015)
+		(start 101.219999 58.679999)
+		(end 100.5 57.96)
 		(width 0.2)
 		(layer "F.Cu")
@@
 	)
 	(segment
-		(start 117 71)
-		(end 130.75 71)
+		(start 119.37 51.25)
+		(end 111.940001 58.679999)
 		(width 0.2)
 		(layer "F.Cu")
-		(net 2)
+		(net 1)
 	)
 	(segment
-		(start 111 63.75)
-		(end 111 65)
+		(start 119.37 51.25)
+		(end 121.985 51.25)
 		(width 0.2)
 		(layer "F.Cu")
-		(net 2)
+		(net 1)
 	)
 	(segment
-		(start 111 57.25)
-		(end 111 63.75)
+		(start 119.37 69.75)
+		(end 121.015 69.75)
 		(width 0.2)
 		(layer "F.Cu")
-		(net 2)
+		(net 1)
 	)
 	(segment
-		(start 111 56)
-		(end 117.97 49.03)
+		(start 111 63.75)
+		(end 118.25 71)
 		(width 0.2)
 		(layer "F.Cu")
@@
 	)
 	(segment
-		(start 111 65)
-		(end 117 71)
+		(start 111 57.25)
+		(end 119.22 49.03)
 		(width 0.2)
 		(layer "F.Cu")
@@
 	)
 	(segment
-		(start 111 57.25)
-		(end 111 56)
+		(start 118.25 71)
+		(end 130.75 71)
 		(width 0.2)
 		(layer "F.Cu")
@@
 	)
 	(segment
-		(start 117.97 49.03)
+		(start 119.22 49.03)
 		(end 130.75 49.03)
 		(width 0.2)
@@
 	)
 	(segment
+		(start 111 57.25)
+		(end 111 63.75)
+		(width 0.2)
+		(layer "B.Cu")
+		(net 2)
+	)
+	(segment
 		(start 105.5 51.25)
 		(end 111.75 51.25)
@@
 	)
 	(segment
-		(start 100.5 64.58)
-		(end 100.5 63.04)
-		(width 0.2)
-		(layer "F.Cu")
-		(net 5)
-	)
-	(segment
-		(start 102.96 53.96)
-		(end 100.5 56.42)
-		(width 0.2)
-		(layer "F.Cu")
-		(net 5)
-	)
-	(segment
-		(start 100.5 56.42)
-		(end 100.5 57.96)
-		(width 0.2)
-		(layer "F.Cu")
-		(net 5)
-	)
-	(segment
-		(start 102.96 51.25)
-		(end 102.96 53.96)
+		(start 99.479 60.5)
+		(end 99.479 54.731)
 		(width 0.2)
 		(layer "F.Cu")
@@
 	(segment
 		(start 102.96 69.75)
-		(end 102.96 67.04)
+		(end 99.479 66.269)
 		(width 0.2)
 		(layer "F.Cu")
@@
 	)
 	(segment
-		(start 103.765 69.75)
-		(end 102.96 69.75)
+		(start 99.479 54.731)
+		(end 102.96 51.25)
 		(width 0.2)
 		(layer "F.Cu")
@@
 	)
 	(segment
-		(start 100.5 63.04)
-		(end 100.5 57.96)
+		(start 103.04 60.5)
+		(end 99.479 60.5)
 		(width 0.2)
 		(layer "F.Cu")
@@
 	)
 	(segment
-		(start 102.96 67.04)
-		(end 100.5 64.58)
+		(start 99.479 66.269)
+		(end 99.479 60.5)
 		(width 0.2)
 		(layer "F.Cu")
@@
 	)
 	(segment
-		(start 103.04 60.5)
-		(end 103.04 62.04)
-		(width 0.2)
-		(layer "F.Cu")
-		(net 6)
-	)
-	(segment
-		(start 103.04 58.96)
-		(end 104.75 57.25)
-		(width 0.2)
-		(layer "F.Cu")
-		(net 6)
-	)
-	(segment
-		(start 104.75 63.75)
+		(start 105.79 63.04)
 		(end 106.5 63.75)
 		(width 0.2)
@@
 	)
 	(segment
-		(start 103.04 62.04)
-		(end 104.75 63.75)
-		(width 0.2)
-		(layer "F.Cu")
-		(net 6)
-	)
-	(segment
-		(start 104.75 57.25)
-		(end 106.5 57.25)
+		(start 100.5 63.04)
+		(end 105.79 63.04)
 		(width 0.2)
 		(layer "F.Cu")
@@
 	)
 	(segment
-		(start 103.04 60.5)
-		(end 103.04 58.96)
+		(start 106.5 57.25)
+		(end 106.5 63.75)
 		(width 0.2)
-		(layer "F.Cu")
+		(layer "B.Cu")
 		(net 6)
 	)
